File: projects/motion-nightlight/motion-nightlight.kicad_pcb (KiCad board)
At the start: 2 copper layers, 47 x 29 mm, 24 parts, among them J1 J_PWR3, Q1 DARK ON, Q2 LED ON, SW1 LAMP TEST, SW2 SENSOR, SW3 MODE, U1 74HC14, U2 74HC08

Commit message: Update motion nightlight PCB and documentation
Parts:
- Q1: value DARK ON -> MMBT3904; footprint Package_TO_SOT_SMD:SOT-23_Handsoldering -> Package_TO_SOT_SMD:SOT-23
- Q2: footprint Package_TO_SOT_SMD:SOT-23_Handsoldering -> Package_TO_SOT_SMD:SOT-23
- RV1: value D TRIM -> DARK TRIM
- RV2: value M TRIM -> MOTION TRIM
- moved Q1 1.25 mm to (124.0, 81.5), turned to 0 degrees
Connections:
- Q1 pad 1: GND -> Net-(Q1-B)
- Q1 pad 2: Net-(Q1-B) -> GND
Routing:
- net Net-(Q1-B): track 10.8 -> 13.8 mm
- net /DARK_RAW: track 12.8 -> 10.9 mm
