File: projects/motion-nightlight/motion-nightlight.kicad_sch (KiCad schematic)
At the start: 24 parts, among them J1 J_PWR3, Q1 DARK ON, Q2 LED ON, SW1 LAMP TEST, SW2 SENSOR, SW3 MODE, U1 74HC14, U2 74HC08

Commit message: Update motion nightlight PCB and documentation
Parts:
- removed Q1: DARK ON, Package_TO_SOT_SMD:SOT-23_Handsoldering, symbol Transistor_BJT:Q_NPN_EBC
- added Q1: MMBT3904, Package_TO_SOT_SMD:SOT-23, symbol Transistor_BJT:MMBT3904
- Q2: footprint Package_TO_SOT_SMD:SOT-23_Handsoldering -> Package_TO_SOT_SMD:SOT-23; symbol Transistor_FET:Q_NMOS_GSD -> Transistor_FET:AO3400A
Connections:
- net DARK_RAW: now also Q1.3 (C)
- net GND: now also Q1.2 (E)
- net at R2.2, R3.2: now also Q1.1 (B)
Changed lines of the file:
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@@
 	)
 	(junction
-		(at 63.5 91.44)
-		(diameter 0)
-		(color 0 0 0 0)
-	)
-	(junction
 		(at 82.55 29.21)
 		(diameter 0)
@@
 	)
 	(junction
+		(at 63.5 91.44)
+		(diameter 0)
+		(color 0 0 0 0)
+	)
+	(junction
 		(at 121.92 116.84)
 		(diameter 0)
@@
 	(wire
 		(pts
-			(xy 63.5 91.44) (xy 92.71 91.44)
+			(xy 215.9 119.38) (xy 215.9 129.54)
 		)
 		(stroke
@@
 	(wire
 		(pts
-			(xy 215.9 119.38) (xy 215.9 129.54)
+			(xy 121.92 116.84) (xy 137.16 116.84)
 		)
 		(stroke
@@
 	(wire
 		(pts
-			(xy 121.92 116.84) (xy 137.16 116.84)
+			(xy 140.97 100.33) (xy 153.67 100.33)
 		)
 		(stroke
@@
 	(wire
 		(pts
-			(xy 140.97 100.33) (xy 153.67 100.33)
+			(xy 66.04 133.35) (xy 76.2 133.35)
 		)
 		(stroke
@@
 	(wire
 		(pts
-			(xy 66.04 133.35) (xy 76.2 133.35)
+			(xy 140.97 116.84) (xy 143.51 116.84)
 		)
 		(stroke
@@
 	(wire
 		(pts
-			(xy 140.97 116.84) (xy 143.51 116.84)
+			(xy 165.1 35.56) (xy 179.07 35.56)
 		)
 		(stroke
@@
 	(wire
 		(pts
-			(xy 165.1 35.56) (xy 179.07 35.56)
+			(xy 66.04 125.73) (xy 66.04 128.27)
 		)
 		(stroke
@@
 	(wire
 		(pts
-			(xy 66.04 125.73) (xy 66.04 128.27)
+			(xy 63.5 91.44) (xy 92.71 91.44)
 		)
 		(stroke
@@
 	)
 	(symbol
-		(lib_name "Q_NPN_EBC_1")
-		(lib_id "Transistor_BJT:Q_NPN_EBC")
-		(at 60.96 86.36 0)
-		(mirror x)
-		(unit 1)
-		(exclude_from_sim no)
-		(in_bom yes)
-		(on_board yes)
-		(dnp no)
-		(property "Reference" "Q1"
-			(at 66.04 87.6301 0)
-			(effects
-				(font
-					(size 1.27 1.27)
-				)
-				(justify left)
-			)
-		)
-		(property "Value" "DARK ON"
-			(at 68.58 86.106 0)
-			(effects
-				(font
-					(size 1.27 1.27)
-				)
-				(justify left)
-			)
-		)
-		(property "Footprint" "Package_TO_SOT_SMD:SOT-23_Handsoldering"
-			(at 66.04 88.9 0)
-			(effects
-				(font
-					(size 1.27 1.27)
-				)
-				(hide yes)
-			)
-		)
-		(property "Datasheet" "~"
-			(at 60.96 86.36 0)
-			(effects
-				(font
-					(size 1.27 1.27)
-				)
-				(hide yes)
-			)
-		)
-		(property "Description" "NPN transistor, emitter/base/collector"
-			(at 60.96 86.36 0)
-			(effects
-				(font
-					(size 1.27 1.27)
-				)
-				(hide yes)
-			)
-		)
-		(pin "3"
-		)
-		(pin "1"
-		)
-		(pin "2"
-		)
-		(instances
-			(project ""
-				(path "/f8cd0c1c-0b03-49c8-b5d7-6c5c8a2c3085"
-					(reference "Q1")
-					(unit 1)
-				)
-			)
-		)
-	)
-	(symbol
 		(lib_id "power:+5V")
 		(at 95.25 31.75 180)
@@
 	)
 	(symbol
-		(lib_id "Transistor_FET:Q_NMOS_GSD")
+		(lib_id "Transistor_BJT:MMBT3904")
+		(at 60.96 86.36 0)
+		(mirror x)
+		(unit 1)
+		(exclude_from_sim no)
+		(in_bom yes)
+		(on_board yes)
+		(dnp no)
+		(property "Reference" "Q1"
+			(at 66.04 87.6301 0)
+			(effects
+				(font
+					(size 1.27 1.27)
+				)
+				(justify left)
+			)
+		)
+		(property "Value" "MMBT3904"
+			(at 66.04 85.0901 0)
+			(effects
+				(font
+					(size 1.27 1.27)
+				)
+				(justify left)
+			)
+		)
+		(property "Footprint" "Package_TO_SOT_SMD:SOT-23"
+			(at 66.04 84.455 0)
+			(effects
+				(font
+					(size 1.27 1.27)
+					(italic yes)
+				)
+				(justify left)
+				(hide yes)
+			)
+		)
+		(property "Datasheet" "https://www.onsemi.com/pdf/datasheet/pzt3904-d.pdf"
+			(at 60.96 86.36 0)
+			(effects
+				(font
+					(size 1.27 1.27)
+				)
+				(justify left)
+				(hide yes)
+			)
+		)
+		(property "Description" "0.2A Ic, 40V Vce, Small Signal NPN Transistor, SOT-23"
+			(at 60.96 86.36 0)
+			(effects
+				(font
+					(size 1.27 1.27)
+				)
+				(hide yes)
+			)
+		)
+		(property "Sim.Device" "NPN"
+			(at 60.96 86.36 0)
+			(effects
+				(font
+					(size 1.27 1.27)
+				)
+				(hide yes)
+			)
+		)
+		(property "Sim.Pins" "1=B 2=E 3=C"
+			(at 60.96 86.36 0)
+			(effects
+				(font
+					(size 1.27 1.27)
+				)
+				(hide yes)
+			)
+		)
+		(pin "2"
+		)
+		(pin "1"
+		)
+		(pin "3"
+		)
+		(instances
+			(project ""
+				(path "/f8cd0c1c-0b03-49c8-b5d7-6c5c8a2c3085"
+					(reference "Q1")
+					(unit 1)
+				)
+			)
+		)
+	)
+	(symbol
+		(lib_id "Transistor_FET:AO3400A")
 		(at 171.45 53.34 0)
 		(unit 1)
@@
 			)
 		)
-		(property "Footprint" "Package_TO_SOT_SMD:SOT-23_Handsoldering"
-			(at 176.53 50.8 0)
+		(property "Footprint" "Package_TO_SOT_SMD:SOT-23"
+			(at 176.53 55.245 0)
 			(effects
 				(font
 					(size 1.27 1.27)
+					(italic yes)
 				)
+				(justify left)
 				(hide yes)
 			)
 		)
-		(property "Datasheet" "~"
-			(at 171.45 53.34 0)
+		(property "Datasheet" "http://www.aosmd.com/pdfs/datasheet/AO3400A.pdf"
+			(at 176.53 57.15 0)
 			(effects
 				(font
 					(size 1.27 1.27)
 				)
+				(justify left)
 				(hide yes)
 			)
 		)
-		(property "Description" "N-MOSFET transistor, gate/source/drain"
+		(property "Description" "30V Vds, 5.7A Id, N-Channel MOSFET, SOT-23"
 			(at 171.45 53.34 0)
 			(effects
